File: PCB/mzdotdiag/DiagOut.kicad_sch (KiCad schematic)
At the start: 24 parts, among them Q1 Q_NPN_BEC, Q2 Q_NPN_BEC, Q3 Q_NPN_BEC, Q4 Q_NPN_BEC, Q5 Q_NPN_BEC, Q6 Q_NPN_BEC, Q7 Q_NPN_BEC, Q8 Q_NPN_BEC

Commit message: Lots of schematic updates, found CD4504B for logic level shifting
Parts:
- Q1, Q2, Q3, Q4, Q5, Q6, Q7, Q8: footprint (none) -> Package_TO_SOT_SMD:SOT-23; LOMEX (none) -> 86-05-65
- R10, R15, R16, R17, R18, R7, R8, R9: footprint (none) -> Resistor_SMD:R_0603_1608Metric
- R11, R12, R13, R14, R3, R4, R5, R6: footprint (none) -> Resistor_SMD:R_0603_1608Metric; LOMEX (none) -> 81-10-26
